File: mx_version/mx_version.kicad_pcb (KiCad board)
At the start: 2 copper layers, 116.9 x 100.3 mm, 78 parts, among them SW1 Switch, SW10 Switch, SW11 Switch, SW12 Switch, SW13 Switch, SW14 Switch, SW15 Switch, SW16 Switch, SW17 Switch, SW18 Switch, SW19 Switch, SW2 Switch, SW20 Switch, SW21 Switch, SW22 Switch, SW23 Switch, SW24 Switch, SW25 Switch, SW26 Switch, SW27 Switch, SW28 Switch, SW29 Switch, SW3 Switch, SW30 Switch, SW31 Switch, SW32 Switch, SW33 Switch, SW34 Switch, SW4 Switch, SW5 Switch, SW6 Switch, SW7 Switch, SW8 Switch, SW9 Switch, U1 XIAO-nRF52840-DIP, U2 XIAO-nRF52840-DIP

Commit message: updated
Parts:
- moved SW37 10.3 mm to (167.8, 75.3)
- moved SW38 10.3 mm to (167.8, 75.3)
- moved SW35 9.73 mm to (167.8, 85.3)
- moved SW36 9.73 mm to (167.8, 85.3)
- moved U1 0.44 mm to (157.7, 56.2)
- moved U2 0.44 mm to (157.7, 56.2)
- renumbered RST to SW35, RST to SW36, POWER to SW37, POWER to SW38, RST to TP1, GND to TP2, RST to TP3, GND to TP4
Connections:
- net PWR_SWITCH_LEFT renamed PWR_SW_LEFT
- net RESET_LEFT renamed RST_LEFT
- net RESET_RIGHT renamed RST_RIGHT
- SW18 pad 1: CR1 -> CR5
- SW19 pad 1: CR1 -> CR5
- SW20 pad 1: CR1 -> CR5
- SW21 pad 1: CR2 -> CR4
- SW22 pad 1: CR2 -> CR4
- SW23 pad 1: CR2 -> CR4
- SW27 pad 1: CR4 -> CR2
- SW28 pad 1: CR4 -> CR2
- SW29 pad 1: CR4 -> CR2
- SW30 pad 1: CR4 -> CR2
- SW31 pad 1: CR5 -> CR1
- SW32 pad 1: CR5 -> CR1
- SW33 pad 1: CR5 -> CR1
- SW34 pad 1: CR5 -> CR1
- SW38 pad 2: PWR_SWITCH_RIGHT -> PWR_SW_RIGHT
- U1 pad 5: CL5 -> RL1
- U1 pad 6: RL1 -> CL5
- U2 pad 1: CR1 -> unconnected-(U2-P0.02_AIN0_LOW_A0_D0-Pad1)_2
- U2 pad 10: PWR_SWITCH_RIGHT -> RR1
- U2 pad 11: unconnected-(U2-P1.15_MOSI_D10-Pad11)_2 -> CR1
- U2 pad 2: CR2 -> PWR_SW_RIGHT
- U2 pad 3: CR3 -> RR4
- U2 pad 4: CR4 -> CR5
- U2 pad 5: CR5 -> CR4
- U2 pad 6: RR1 -> RR3
- U2 pad 7: RR2 -> CR3
- U2 pad 8: RR3 -> RR2
- U2 pad 9: RR4 -> CR2
Routing:
- net CR5: track 0.00 -> 186.4 mm, vias 0 -> 2
- net CR4: track 0.00 -> 169.5 mm, vias 0 -> 2
- net RL3: track 0.00 -> 141.3 mm, vias 0 -> 4
- net CL1: track 0.00 -> 141.0 mm, vias 0 -> 6
- net RR3: track 0.00 -> 140.8 mm, vias 0 -> 8
- net CL2: track 0.00 -> 123.4 mm, vias 0 -> 2
- net GND: track 0.00 -> 121.4 mm, vias 0 -> 43
- net RR2: track 0.00 -> 111.4 mm, vias 0 -> 10
- net RL2: track 0.00 -> 111.2 mm, vias 0 -> 8
- net CR3: track 0.00 -> 109.0 mm, vias 0 -> 4
- net RR4: track 0.00 -> 105.9 mm
- net CL3: track 0.00 -> 103.6 mm, vias 0 -> 2
- net CL4: track 0.00 -> 101.9 mm, vias 0 -> 2
- net RL1: track 0.00 -> 101.3 mm, vias 0 -> 8
- net RL4: track 0.00 -> 99.0 mm
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- added copper zone on B.Cu, net GND
- added copper zone on F.Cu, net GND
Other:
- board size 116.9 x 100.3 mm -> 116.9 x 99.9 mm
