File: mx_version/mx_version.kicad_sch (KiCad schematic)
At the start: 78 parts, among them SW1 Switch, SW10 Switch, SW11 Switch, SW12 Switch, SW13 Switch, SW14 Switch, SW15 Switch, SW16 Switch, SW17 Switch, SW18 Switch, SW19 Switch, SW2 Switch, SW20 Switch, SW21 Switch, SW22 Switch, SW23 Switch, SW24 Switch, SW25 Switch, SW26 Switch, SW27 Switch, SW28 Switch, SW29 Switch, SW3 Switch, SW30 Switch, SW31 Switch, SW32 Switch, SW33 Switch, SW34 Switch, SW35 Switch, SW36 Switch, SW37 Switch, SW38 Switch, SW4 Switch, SW5 Switch, SW6 Switch, SW7 Switch, SW8 Switch, SW9 Switch, U1 XIAO-nRF52840-DIP, U2 XIAO-nRF52840-DIP

Commit message: updated
Connections:
- net CL5: now also U1.6 (P0.05_AIN3_A5_D5); no longer U1.5 (P0.04_AIN2_A4_D4)
- net CR1: now also SW31.1, SW32.1, SW33.1, SW34.1, U2.11 (P1.15_MOSI_D10); no longer SW18.1, SW19.1, SW20.1, U2.1 (P0.02_AIN0_LOW_A0_D0)
- net CR2: now also SW27.1, SW28.1, SW29.1, SW30.1, U2.9 (P1.13_SCK_D8); no longer SW21.1, SW22.1, SW23.1, U2.2 (P0.03_AIN1_LOW_A1_D1)
- net CR3: now also U2.7 (P1.11_TX_D6); no longer U2.3 (P0.28_AIN4_LOW_A2_D2)
- net CR4: now also SW21.1, SW22.1, SW23.1, U2.5 (P0.04_AIN2_A4_D4); no longer SW27.1, SW28.1, SW29.1, SW30.1, U2.4 (P0.29_AIN5_LOW_A3_D3)
- net CR5: now also SW18.1, SW19.1, SW20.1, U2.4 (P0.29_AIN5_LOW_A3_D3); no longer SW31.1, SW32.1, SW33.1, SW34.1, U2.5 (P0.04_AIN2_A4_D4)
- net RL1: now also U1.5 (P0.04_AIN2_A4_D4); no longer U1.6 (P0.05_AIN3_A5_D5)
- net RR1: now also U2.10 (P1.14_MISO_D9); no longer U2.6 (P0.05_AIN3_A5_D5)
- net RR2: now also U2.8 (P1.12_RX_D7); no longer U2.7 (P1.11_TX_D6)
- net RR3: now also U2.6 (P0.05_AIN3_A5_D5); no longer U2.8 (P1.12_RX_D7)
- net RR4: now also U2.3 (P0.28_AIN4_LOW_A2_D2); no longer U2.9 (P1.13_SCK_D8)
- net PWR_SWITCH_LEFT renamed PWR_SW_LEFT
- net PWR_SWITCH_RIGHT renamed PWR_SW_RIGHT
- net PWR_SW_RIGHT: now also U2.2 (P0.03_AIN1_LOW_A1_D1); no longer U2.10 (P1.14_MISO_D9)
- net RESET_LEFT renamed RST_LEFT
- net RESET_RIGHT renamed RST_RIGHT
Other:
- moved on the sheet: TP2, TP4
