File: mx_nrfpromicro/mx_nrfpromicro.kicad_pcb (KiCad board)
At the start: 2 copper layers, 0 parts

Commit message: updated
Parts:
- added SW1: SW_Push_45deg, BLE_KBD:MX_Optional_Reversible_1u, F.Cu at (311.6, 20.7)
- added SW10: SW_Push_45deg, BLE_KBD:MX_Optional_Reversible_1u, F.Cu at (330.2, 66.1)
- added SW11: SW_Push_45deg, BLE_KBD:MX_Optional_Reversible_1u, F.Cu at (330.2, 81.3)
- added SW12: SW_Push_45deg, BLE_KBD:MX_Optional_Reversible_1u, F.Cu at (330.2, 96.4)
- added SW13: SW_Push_45deg, BLE_KBD:MX_Optional_Reversible_1u, F.Cu at (348.9, 20.7)
- added SW14: SW_Push_45deg, BLE_KBD:MX_Optional_Reversible_1u, F.Cu at (348.9, 35.8)
- added SW15: SW_Push_45deg, BLE_KBD:MX_Optional_Reversible_1u, F.Cu at (348.9, 51.0)
- added SW16: SW_Push_45deg, BLE_KBD:MX_Optional_Reversible_1.5u, F.Cu at (348.9, 66.1)
- added SW17: SW_Push_45deg, BLE_KBD:MX_Optional_Reversible_1.5u, F.Cu at (348.9, 81.3)
- added SW18: ~, BLE_KBD:SS12F23G5, F.Cu at (384.3, 61.2)
- added SW19: ~, BLE_KBD:SW_SIDE_MOUNT, F.Cu at (385.4, 73.8)
- added SW2: SW_Push_45deg, BLE_KBD:MX_Optional_Reversible_1u, F.Cu at (311.6, 35.8)
- added SW3: SW_Push_45deg, BLE_KBD:MX_Optional_Reversible_1u, F.Cu at (311.6, 51.0)
- added SW4: SW_Push_45deg, BLE_KBD:MX_Optional_Reversible_1u, F.Cu at (311.6, 66.1)
- added SW5: SW_Push_45deg, BLE_KBD:MX_Optional_Reversible_1u, F.Cu at (311.6, 81.3)
- added SW6: SW_Push_45deg, BLE_KBD:MX_Optional_Reversible_1u, F.Cu at (311.6, 96.4)
- added SW7: SW_Push_45deg, BLE_KBD:MX_Optional_Reversible_1u, F.Cu at (330.2, 20.7)
- added SW8: SW_Push_45deg, BLE_KBD:MX_Optional_Reversible_1u, F.Cu at (330.2, 35.8)
- added SW9: SW_Push_45deg, BLE_KBD:MX_Optional_Reversible_1u, F.Cu at (330.2, 51.0)
- added TP1: TestPoint_Small, TestPoint:TestPoint_THTPad_D1.0mm_Drill0.5mm, F.Cu at (369.7, 62.6)
- added TP2: TestPoint_Small, TestPoint:TestPoint_THTPad_D1.0mm_Drill0.5mm, F.Cu at (369.7, 65.6)
- added U1: Nice_Nano_V2, BLE_KBD:Nice_Nano_V2, F.Cu at (368.0, 31.5)
