File: mx_nrfpromicro/mx_nrfpromicro.kicad_sch (KiCad schematic)
At the start: 21 parts, among them J1 Conn_01x02, SW1 SW_Push_45deg, SW10 SW_Push_45deg, SW11 SW_Push_45deg, SW12 SW_Push_45deg, SW13 SW_Push_45deg, SW14 SW_Push_45deg, SW15 SW_Push_45deg, SW16 SW_Push_45deg, SW17 SW_Push_45deg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

Commit message: updated
Parts:
- added S2: EG1215AA, EG1215AA:SW_EG1215AA, symbol EG1215AA:EG1215AA
Connections:
- net at S1.2, U1.24 (B+): now also S2.2
- net at J1.1 (Pin_1), S1.1: now also S2.1
- no-connect marks 3 -> 4
Other:
- moved on the sheet: J1, S1, SW18, U1

Commit message: updated
Parts:
- removed J1: Conn_01x02, symbol Connector_Generic:Conn_01x02
- removed S1, S2: EG1215AA, EG1215AA:SW_EG1215AA, symbol EG1215AA:EG1215AA
- removed SW18: SW_Push, symbol Switch:SW_Push
- added PWR_SW: ~, BLE_KBD:SS12F23G5, symbol SS12F23G5:SS12F23G5
- added RST: ~, BLE_KBD:SW_SIDE_MOUNT, symbol SW_SIDE_MOUNT:SW_SIDE_MOUNT
- added TP1, TP2: TestPoint_Small, TestPoint:TestPoint_THTPad_D1.0mm_Drill0.5mm, symbol Connector:TestPoint_Small
- SW1, SW10, SW11, SW12, SW13, SW14, SW15, SW2, SW3, SW4, SW5, SW6, SW7, SW8, SW9: footprint (none) -> BLE_KBD:MX_Optional_Reversible_1u
- SW16, SW17: footprint (none) -> BLE_KBD:MX_Optional_Reversible_1.5u
- U1: footprint ScottoKeebs_MCU:Nice_Nano_V2 -> BLE_KBD:Nice_Nano_V2
Connections:
- net GND: now also PWR_SW.4, PWR_SW.5, RST.2, RST.3, RST.4, TP2.1
- net RST: now also RST.1
- net at U1.24 (B+): now also PWR_SW.1
- new net: PWR_SW.2, TP1.1
- no-connect marks 4 -> 3
Other:
- moved on the sheet: SW1, SW10, SW11, SW12, SW13, SW14, SW15, SW16, SW17, SW2, SW3, SW4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

Commit message: updated
Parts:
- removed PWR_SW: ~, BLE_KBD:SS12F23G5, symbol SS12F23G5:SS12F23G5
- removed RST: ~, BLE_KBD:SW_SIDE_MOUNT, symbol SW_SIDE_MOUNT:SW_SIDE_MOUNT
- added SW18: SW_SPDT, BLE_KBD:SS12F23G5, symbol SS12F23G5:SS12F23G5
- added SW19: SW_PUSH, BLE_KBD:SW_SIDE_MOUNT, symbol SW_SIDE_MOUNT:SW_SIDE_MOUNT
Connections:
- net GND: now also SW18.4, SW18.5, SW19.2, SW19.3, SW19.4
- net RST: now also SW19.1
- net at U1.24 (B+): now also SW18.1
- net at TP1.1: now also SW18.2
Changed lines of the file:
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@@
 	(paper "A4")
 	(junction
-		(at 138.43 80.01)
-		(diameter 0)
-		(color 0 0 0 0)
-	)
-	(junction
 		(at 162.56 35.56)
 		(diameter 0)
@@
 		(color 0 0 0 0)
 	)
+	(junction
+		(at 138.43 80.01)
+		(diameter 0)
+		(color 0 0 0 0)
+	)
 	(no_connect
 		(at 154.94 43.18)
@@
 	(wire
 		(pts
-			(xy 138.43 74.93) (xy 138.43 80.01)
+			(xy 114.3 41.91) (xy 114.3 40.64)
 		)
 		(stroke
@@
 	(wire
 		(pts
-			(xy 114.3 41.91) (xy 114.3 40.64)
+			(xy 154.94 40.64) (xy 153.67 40.64)
 		)
 		(stroke
@@
 	(wire
 		(pts
-			(xy 154.94 40.64) (xy 153.67 40.64)
+			(xy 158.75 19.05) (xy 158.75 20.32)
 		)
 		(stroke
@@
 	(wire
 		(pts
-			(xy 158.75 19.05) (xy 158.75 20.32)
+			(xy 156.21 33.02) (xy 153.67 33.02)
 		)
 		(stroke
@@
 	(wire
 		(pts
-			(xy 156.21 33.02) (xy 153.67 33.02)
+			(xy 138.43 74.93) (xy 138.43 80.01)
 		)
 		(stroke
@@
 	)
 	(symbol
-		(lib_id "Switch:SW_Push_45deg")
-		(at 96.52 22.86 0)
+		(lib_id "SW_SIDE_MOUNT:SW_SIDE_MOUNT")
+		(at 133.35 77.47 0)
 		(unit 1)
 		(exclude_from_sim no)
@@
 		(dnp no)
 		(fields_autoplaced yes)
-		(property "Reference" "SW5"
-			(at 96.52 15.24 0)
+		(property "Reference" "SW19"
+			(at 133.35 68.58 0)
 			(effects
 				(font
@@
 			)
 		)
-		(property "Value" "SW_Push_45deg"
-			(at 96.52 17.78 0)
+		(property "Value" "SW_PUSH"
+			(at 133.35 71.12 0)
 			(effects
 				(font
@@
 			)
 		)
-		(property "Footprint" "BLE_KBD:MX_Optional_Reversible_1u"
-			(at 96.52 22.86 0)
+		(property "Footprint" "BLE_KBD:SW_SIDE_MOUNT"
+			(at 133.35 77.47 0)
 			(effects
 				(font
@@
 			)
 		)
-		(property "Datasheet" "~"
-			(at 96.52 22.86 0)
+		(property "Datasheet" ""
+			(at 133.35 77.47 0)
 			(effects
 				(font
@@
 			)
 		)
-		(property "Description" "Push button switch, normally open, two pins, 45° tilted"
-			(at 96.52 22.86 0)
+		(property "Description" ""
+			(at 133.35 77.47 0)
 			(effects
 				(font
@@
 		(pin "2"
 		)
+		(pin "3"
+		)
+		(pin "4"
+		)
 		(instances
-			(project "mx_nrfpromicro"
+			(project ""
 				(path "/ce115848-5daa-4079-937d-d5b781bb7914"
-					(reference "SW5")
+					(reference "SW19")
 					(unit 1)
 				)
@@
 	)
 	(symbol
-		(lib_id "power:GND")
-		(at 27.94 25.4 0)
+		(lib_id "Switch:SW_Push_45deg")
+		(at 96.52 22.86 0)
 		(unit 1)
 		(exclude_from_sim no)
@@
 		(dnp no)
 		(fields_autoplaced yes)
-		(property "Reference" "#PWR02"
-			(at 27.94 31.75 0)
+		(property "Reference" "SW5"
+			(at 96.52 15.24 0)
 			(effects
 				(font
 					(size 1.27 1.27)
 				)
-				(hide yes)
 			)
 		)
-		(property "Value" "GND"
-			(at 27.94 30.48 0)
+		(property "Value" "SW_Push_45deg"
+			(at 96.52 17.78 0)
 			(effects
 				(font
@@
 			)
 		)
-		(property "Footprint" ""
-			(at 27.94 25.4 0)
+		(property "Footprint" "BLE_KBD:MX_Optional_Reversible_1u"
+			(at 96.52 22.86 0)
 			(effects
 				(font
@@
 			)
 		)
-		(property "Datasheet" ""
-			(at 27.94 25.4 0)
+		(property "Datasheet" "~"
+			(at 96.52 22.86 0)
 			(effects
 				(font
@@
 			)
 		)
-		(property "Description" "Power symbol creates a global label with name \"GND\" , ground"
-			(at 27.94 25.4 0)
+		(property "Description" "Push button switch, normally open, two pins, 45° tilted"
+			(at 96.52 22.86 0)
 			(effects
 				(font
@@
 		(pin "1"
 		)
+		(pin "2"
+		)
 		(instances
-			(project ""
+			(project "mx_nrfpromicro"
 				(path "/ce115848-5daa-4079-937d-d5b781bb7914"
-					(reference "#PWR02")
+					(reference "SW5")
 					(unit 1)
 				)
@@
 	(symbol
 		(lib_id "power:GND")
-		(at 81.28 44.45 0)
+		(at 27.94 25.4 0)
 		(unit 1)
 		(exclude_from_sim no)
@@
 		(dnp no)
 		(fields_autoplaced yes)
-		(property "Reference" "#PWR012"
-			(at 81.28 50.8 0)
+		(property "Reference" "#PWR02"
+			(at 27.94 31.75 0)
 			(effects
 				(font
@@
 		)
 		(property "Value" "GND"
-			(at 81.28 49.53 0)
+			(at 27.94 30.48 0)
 			(effects
 				(font
@@
 		)
 		(property "Footprint" ""
-			(at 81.28 44.45 0)
+			(at 27.94 25.4 0)
 			(effects
 				(font
@@
 		)
 		(property "Datasheet" ""
-			(at 81.28 44.45 0)
+			(at 27.94 25.4 0)
 			(effects
 				(font
@@
 		)
 		(property "Description" "Power symbol creates a global label with name \"GND\" , ground"
-			(at 81.28 44.45 0)
+			(at 27.94 25.4 0)
 			(effects
 				(font
@@
 		)
 		(instances
-			(project "mx_nrfpromicro"
+			(project ""
 				(path "/ce115848-5daa-4079-937d-d5b781bb7914"
-					(reference "#PWR012")
+					(reference "#PWR02")
 					(unit 1)
 				)
@@
 	)
 	(symbol
-		(lib_id "SS12F23G5:SS12F23G5")
-		(at 158.75 25.4 90)
+		(lib_id "power:GND")
+		(at 81.28 44.45 0)
 		(unit 1)
 		(exclude_from_sim no)
@@
 		(dnp no)
 		(fields_autoplaced yes)
-		(property "Reference" "PWR_SW"
-			(at 163.83 24.7649 90)
+		(property "Reference" "#PWR012"
+			(at 81.28 50.8 0)
 			(effects
 				(font
 					(size 1.27 1.27)
 				)
-				(justify right)
+				(hide yes)
 			)
 		)
-		(property "Value" "~"
-			(at 163.83 26.67 90)
+		(property "Value" "GND"
+			(at 81.28 49.53 0)
 			(effects
 				(font
 					(size 1.27 1.27)
 				)
-				(justify right)
 			)
 		)
-		(property "Footprint" "BLE_KBD:SS12F23G5"
-			(at 158.75 25.4 0)
+		(property "Footprint" ""
+			(at 81.28 44.45 0)
 			(effects
 				(font
@@
 		)
 		(property "Datasheet" ""
-			(at 158.75 25.4 0)
+			(at 81.28 44.45 0)
 			(effects
 				(font
@@
 			)
 		)
-		(property "Description" ""
-			(at 158.75 25.4 0)
+		(property "Description" "Power symbol creates a global label with name \"GND\" , ground"
+			(at 81.28 44.45 0)
 			(effects
 				(font
@@
 			)
 		)
-		(pin "3"
-		)
-		(pin "5"
-		)
 		(pin "1"
 		)
-		(pin "4"
-		)
-		(pin "2"
-		)
 		(instances
-			(project ""
+			(project "mx_nrfpromicro"
 				(path "/ce115848-5daa-4079-937d-d5b781bb7914"
-					(reference "PWR_SW")
+					(reference "#PWR012")
 					(unit 1)
 				)
@@
 	)
 	(symbol
+		(lib_id "SS12F23G5:SS12F23G5")
+		(at 158.75 25.4 90)
+		(unit 1)
+		(exclude_from_sim no)
+		(in_bom yes)
+		(on_board yes)
+		(dnp no)
+		(fields_autoplaced yes)
+		(property "Reference" "SW18"
+			(at 163.83 24.1299 90)
+			(effects
+				(font
+					(size 1.27 1.27)
+				)
+				(justify right)
+			)
+		)
+		(property "Value" "SW_SPDT"
+			(at 163.83 26.6699 90)
+			(effects
+				(font
+					(size 1.27 1.27)
+				)
+				(justify right)
+			)
+		)
+		(property "Footprint" "BLE_KBD:SS12F23G5"
+			(at 158.75 25.4 0)
+			(effects
+				(font
+					(size 1.27 1.27)
+				)
+				(hide yes)
+			)
+		)
+		(property "Datasheet" ""
+			(at 158.75 25.4 0)
+			(effects
+				(font
+					(size 1.27 1.27)
+				)
+				(hide yes)
+			)
+		)
+		(property "Description" ""
+			(at 158.75 25.4 0)
+			(effects
+				(font
+					(size 1.27 1.27)
+				)
+				(hide yes)
+			)
+		)
+		(pin "1"
+		)
+		(pin "2"
+		)
+		(pin "3"
+		)
+		(pin "4"
+		)
+		(pin "5"
+		)
+		(instances
+			(project ""
+				(path "/ce115848-5daa-4079-937d-d5b781bb7914"
+					(reference "SW18")
+					(unit 1)
+				)
+			)
+		)
+	)
+	(symbol
 		(lib_id "Connector:TestPoint_Small")
 		(at 166.37 33.02 0)
@@
 					(unit 1)
 				)
-			)
-		)
-	)
-	(symbol
-		(lib_id "SW_SIDE_MOUNT:SW_SIDE_MOUNT")
-		(at 133.35 77.47 0)
-		(unit 1)
-		(exclude_from_sim no)
-		(in_bom yes)
-		(on_board yes)
-		(dnp no)
-		(property "Reference" "RST"
-			(at 133.35 72.136 0)
-			(effects
-				(font
-					(size 1.27 1.27)
-				)
-			)
-		)
-		(property "Value" "~"
-			(at 133.35 72.39 0)
-			(effects
-				(font
-					(size 1.27 1.27)
-				)
-			)
-		)
-		(property "Footprint" "BLE_KBD:SW_SIDE_MOUNT"
-			(at 133.35 77.47 0)
-			(effects
-				(font
-					(size 1.27 1.27)
-				)
-				(hide yes)
-			)
-		)
-		(property "Datasheet" ""
-			(at 133.35 77.47 0)
-			(effects
-				(font
-					(size 1.27 1.27)
-				)
-				(hide yes)
-			)
-		)
-		(property "Description" ""
-			(at 133.35 77.47 0)
-			(effects
-				(font
-					(size 1.27 1.27)
-				)
-				(hide yes)
-			)
-		)
-		(pin "3"
-		)
-		(pin "2"
-		)
-		(pin "4"
-		)
-		(pin "1"
-		)
-		(instances
-			(project ""
-				(path "/ce115848-5daa-4079-937d-d5b781bb7914"
-					(reference "RST")
-					(unit 1)
-				)

Commit message: updated
Parts:
- removed SW18: SW_SPDT, BLE_KBD:SS12F23G5, symbol SS12F23G5:SS12F23G5
- removed SW19: SW_PUSH, BLE_KBD:SW_SIDE_MOUNT, symbol SW_SIDE_MOUNT:SW_SIDE_MOUNT
- added S1, S2: 436331045822, BLE_KBD:4363X10458XX, symbol 436331045822:436331045822
- added SW18, SW19: MLL1200S, BLE_KBD:SW_MLL1200S, symbol MLL1200S:MLL1200S
- SW1, SW10, SW11, SW12, SW13, SW14, SW15, SW2, SW3, SW4, SW5, SW6, SW7, SW8, SW9: footprint BLE_KBD:MX_Optional_Reversible_1u -> BLE_KBD:MX_Reversible_Optional_1u
- SW16, SW17: footprint BLE_KBD:MX_Optional_Reversible_1.5u -> BLE_KBD:MX_Reversible_Optional_1.5u
- TP1: renamed from TP2; footprint TestPoint:TestPoint_THTPad_D1.0mm_Drill0.5mm -> TestPoint:TestPoint_THTPad_D1.5mm_Drill0.7mm
- TP2: renamed from TP1; footprint TestPoint:TestPoint_THTPad_D1.0mm_Drill0.5mm -> TestPoint:TestPoint_THTPad_D1.5mm_Drill0.7mm
Connections:
- net GND: now also S1.2, S1.4, S2.2, S2.4, SW18.G1 (GND), SW18.G2 (GND), SW18.G3 (GND), SW18.G4 (GND), SW19.G1 (GND), SW19.G2 (GND), SW19.G3 (GND), SW19.G4 (GND)
- net RST: now also S1.1, S1.3, S2.1, S2.3
- net SW1: now also U1.17 (18); no longer U1.1
- net SW10: now also U1.5 (2); no longer U1.12 (9)
- net SW11: now also U1.15 (14); no longer U1.13 (10)
- net SW12: now also U1.18 (19); no longer U1.14 (16)
- net SW13: now also U1.12 (9); no longer U1.15 (14)
- net SW14: now also U1.11 (8); no longer U1.16 (15)
- net SW15: now also U1.10 (7); no longer U1.17 (18)
- net SW16: now also U1.14 (16); no longer U1.18 (19)
- net SW17: now also U1.13 (10); no longer U1.19 (20)
- net SW2: now also U1.9 (6); no longer U1.2 (0)
- net SW3: now also U1.7 (4); no longer U1.5 (2)
- net SW4: now also U1.2 (0); no longer U1.6 (3)
- net SW5: now also U1.1; no longer U1.7 (4)
- net SW6: now also U1.16 (15); no longer U1.8 (5)
- net SW7: now also U1.19 (20); no longer U1.9 (6)
- net SW8: now also U1.8 (5); no longer U1.10 (7)
- net SW9: now also U1.6 (3); no longer U1.11 (8)
- net B+: now reaches U1.24 (B+)
- net B+: now also SW18.2, SW19.2
- net at TP2.1: now also SW18.3, SW19.1
- no-connect marks 3 -> 4
Other:
- moved on the sheet: TP1, TP2

Commit message: updated
Parts:
- added H1, H2, H3, H4: MountingHole, MountingHole:MountingHole_2.2mm_M2, symbol Mechanical:MountingHole
- added JP1, JP10, JP11, JP12, JP13, JP16, JP17, JP2, JP20, JP3, JP4, JP5, JP6, JP7, JP8, JP9: SolderJumper_2_Open, BLE_KBD:Solder_Jumper, symbol Jumper:SolderJumper_2_Open
- TP1, TP2: footprint TestPoint:TestPoint_THTPad_D1.5mm_Drill0.7mm -> BLE_KBD:Test_Point
Connections:
- net B+: now also JP2.1 (A), JP3.1 (A); no longer U1.24 (B+)
- net GND: now also JP12.1 (A), JP13.1 (A), JP16.1 (A), JP5.1 (A), JP8.1 (A), JP9.1 (A); no longer SW18.G1 (GND), SW18.G2 (GND), SW18.G3 (GND), SW18.G4 (GND), SW19.G1 (GND), SW19.G2 (GND), SW19.G3 (GND), SW19.G4 (GND), U1.23 (GND), U1.3 (GND), U1.4 (GND)
- net RST: now also JP10.1 (A), JP11.1 (A); no longer U1.22 (RST)
- net SW10: now also JP17.1 (A), JP20.1 (A); no longer U1.5 (2)
- net SW4: now also JP6.1 (A), JP7.1 (A); no longer U1.2 (0)
- net SW5: now also JP1.1 (A), JP4.1 (A); no longer U1.1
- net 20: now reaches U1.20 (21)
- net 20: now also JP20.2 (B)
- net 21: now reaches U1.21 (3.3v)
- net 21: now also JP16.2 (B)
- new net: SW19.G1 (GND), SW19.G2 (GND), SW19.G3 (GND), SW19.G4 (GND)
- new net: SW18.G1 (GND), SW18.G2 (GND), SW18.G3 (GND), SW18.G4 (GND)
- new net 1: JP1.2 (B), JP2.2 (B), U1.1
- new net 2: JP7.2 (B), JP8.2 (B), U1.2 (0)
- new net 22: JP11.2 (B), JP12.2 (B), U1.22 (RST)
- new net 23: JP5.2 (B), JP6.2 (B), U1.23 (GND)
- new net 24: JP3.2 (B), JP4.2 (B), U1.24 (B+)
- new net 3: JP10.2 (B), JP9.2 (B), U1.3 (GND)
- new net 4: JP13.2 (B), U1.4 (GND)
- new net 5: JP17.2 (B), U1.5 (2)
Other:
- moved on the sheet: TP1
